Commit message: Adding support for XACRO and RViz configuration

File: urdf/workcell.xacro (robot description, xacro)
@@ -1,4 +1,6 @@
 <?xml version="1.0" ?>
 <robot name="myworkcell" xmlns:xacro="http://ros.org/wiki/xacro">
+    <xacro:include filename="$(find ur_description)/urdf/ur5.urdf.xacro" />
+    <xacro:ur5_robot prefix="" joint_limited="true"/>
     <link name="world"/>
     <link name="table">
@@ -14,4 +16,9 @@
       </collision>
     </link>
+    <joint name="table_to_robot" type="fixed">
+  	<parent link="table"/>
+ 	<child link="base_link"/>
+  	<origin xyz="0 0 0" rpy="0 0 0"/>
+    </joint>
     <link name="camera_frame"/>
     <joint name="world_to_table" type="fixed">
